File: feinstaub.kicad_pcb (KiCad board)
At the start: 2 copper layers, 67.1 x 62.2 mm, 14 parts, among them J1 Conn_01x04, J2 Conn_01x04, J3 Conn_01x02, SW1 SW_DIP_x01, U1 ESP-12F, U2 bme280_module, U3 AMS1117-3.3

Commit message: update
Routing:
- net SCL: track 71.7 -> 83.5 mm
- net VCC: track 13.7 -> 24.3 mm
- net SDS_RX: track 37.3 -> 40.3 mm
- net +3V3: track 124.8 -> 124.1 mm

Commit message: small update
Other:
- net class Default removed
- net class Power removed
